File: LCD-50-bias-supply.kicad_pcb (KiCad board)
At the start: 2 copper layers, 86.2 x 60.9 mm, 56 parts, among them J1 Conn_01x40_MountingPin, J2 Conn_01x50_MountingPin, J3 Conn_01x50_MountingPin, J4 Conn_01x02, Q1 BC857, Q2 BC850, U1 TPS61085PW, U2 LM7381

Commit message: Changes zener to SOT-23 package, add jobset, generate fabrication file, First release sending to JLCPCB
Parts:
- removed D1, D6: D_Schottky, Diode_SMD:D_SOD-123
- added D12: BZX84Cxx, Package_TO_SOT_SMD:SOT-23, F.Cu at (175.7, 95.0)
- added D13: BZX84Cxx, Package_TO_SOT_SMD:SOT-23, F.Cu at (171.0, 95.2)
- added TP11: TestPoint, TestPoint:TestPoint_Pad_D1.5mm, F.Cu at (178.7, 101.0)
- D3: footprint Diode_SMD:D_SOD-123 -> Diode_SMD:D_SOD-123F
- J2, J3: footprint Connector_FFC-FPC:Molex_54132-5033_1x50-1MP_P0.5mm_Horizontal -> XF2M_5015_1A:CON50_1X50_DRB_XF2C_TYC
- U2: value LM7381 -> LM7321
- moved C1 0.77 mm to (175.7, 88.4)
- moved Q1 0.77 mm to (175.7, 91.3)
- moved C14 0.76 mm to (170.9, 88.3)
- moved Q2 0.76 mm to (171.0, 91.3)
- moved D3 0.25 mm to (142.5, 114.0)
- turned J2 to 0 degrees
- turned J3 to 0 degrees
Routing:
- net GND: track 44.8 -> 55.4 mm, vias 37 -> 86
- net VGH: track 28.3 -> 20.1 mm
- net Net-(D2-A): track 12.7 -> 18.5 mm
- net Net-(D4-K): track 17.5 -> 19.8 mm
- net LED_A: track 130.1 -> 131.4 mm
- net LED_K: track 139.1 -> 140.3 mm
- net /DITHB: track 59.0 -> 58.1 mm
- net VGL: track 25.6 -> 24.8 mm
- net AVDD: track 92.6 -> 91.8 mm
- net VCOM: track 93.2 -> 94.0 mm
- net /LCD_G4: track 111.1 -> 110.3 mm
- net /LCD_R7: track 111.6 -> 110.8 mm
- net /LCD_G7: track 111.1 -> 110.3 mm
- net /VSYNC: track 120.4 -> 119.6 mm
- net /LCD_G2: track 111.1 -> 110.3 mm
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Other:
- board text added: "-AVDD"

Commit message: Finished, 1st PCB order to JLCPCB
Parts:
- C1, C14: value 2.2uF/50V -> 1uF/50V
- C10, C13, C2: value 10uF -> 10uF/25V
- C11, C12, C4: value 1uF/50V -> 470nF/50V
- C3: value 1uF -> 1uF/25V
- D12: value BZX84Cxx -> BZX84C7V5
- D13: value BZX84Cxx -> BZX84C16
- R6: value 1K -> 1.6K
- moved R6 0.18 mm to (171.1, 97.7)
Routing:
- net VGH: track 20.1 -> 27.5 mm
- net VDD: track 136.4 -> 138.9 mm
- net GND: track 55.4 -> 55.6 mm, vias 86 -> 84
Other:
- board size 86.2 x 60.9 mm -> 86.2 x 63.1 mm
