File: LCD-50-bias-supply.kicad_sch (KiCad schematic)
At the start: 17 parts, among them J1 Conn_01x50_MountingPin

Commit message: Change bias supply IC to TPS61085, Finished tracks, TODO: Assigned B.O.M, add more grounding vias
Parts:
- removed C4: 0.47uF/25V, symbol Device:C
- removed D3: BAT54S, Package_TO_SOT_SMD:SOT-23, symbol Diode:BAT54S
- removed R1: 1K, symbol Device:R_Small
- removed R6: 0R, symbol Device:R_Small
- added C10, C13, C2: 10uF, Capacitor_SMD:C_0805_2012Metric, symbol Device:C
- added C12: 1uF/50V, Capacitor_SMD:C_0805_2012Metric, symbol Device:C
- added C15, C5: 100nF/25V, Capacitor_SMD:C_0603_1608Metric, symbol Device:C
- added C16: 1uF/25V, Capacitor_SMD:C_0805_2012Metric, symbol Device:C
- added C17, C18, C19, C24, C25: 2.2uF, Capacitor_SMD:C_0805_2012Metric, symbol Device:C
- added C20: 22pF, Capacitor_SMD:C_0603_1608Metric, symbol Device:C_Small
- added C21, C22, C23, C26, C27, C28: 4.7uF, Capacitor_SMD:C_0805_2012Metric, symbol Device:C
- added C29: 220nF, Capacitor_SMD:C_0603_1608Metric, symbol Device:C_Small
- added C3, C30: 1uF, Capacitor_SMD:C_0805_2012Metric, symbol Device:C
- added C6, C9: 100nF/50V, Capacitor_SMD:C_0603_1608Metric, symbol Device:C
- added C7: 1.1nF/25V, Capacitor_SMD:C_0603_1608Metric, symbol Device:C
- added D10, D3, D8, D9: MBR0520, Diode_SMD:D_SOD-123, symbol Diode:MBR0520
- added D11: MBR0540, Diode_SMD:D_SOD-123, symbol Diode:MBR0540
- added D2, D5: BAT54S, Package_TO_SOT_SMD:SOT-23, symbol Diode:BAT54S
- added D7: 1N5819, Diode_SMD:D_SOD-123, symbol Diode:1N5819
- added J1: Conn_01x40_MountingPin, Connector_FFC-FPC:Omron_XF2M-4015-1A_1x40-1MP_P0.5mm_Horizontal, symbol Connector_Generic_MountingPin:Conn_01x40_MountingPin
- added J2: Conn_01x50_MountingPin, Connector_FFC-FPC:Molex_54132-5033_1x50-1MP_P0.5mm_Horizontal, symbol Connector_Generic_MountingPin:Conn_01x50_MountingPin
- added J4: Conn_01x02, Connector_PinHeader_2.54mm:PinHeader_1x02_P2.54mm_Vertical, symbol Connector_Generic:Conn_01x02
- added JP1, JP10, JP11, JP2, JP3, JP4, JP5, JP6, JP7, JP8, JP9: JMP, Jumper:SolderJumper-2_P1.3mm_Open_RoundedPad1.0x1.5mm, symbol Jumper:SolderJumper_2_Open
- added JP12, JP13, JP14, JP15, JP16: JMP, Jumper:SolderJumper-3_P1.3mm_Open_RoundedPad1.0x1.5mm_NumberLabels, symbol Jumper:SolderJumper_3_Open
- added L1: 3.3uH, Inductor_SMD:L_Abracon_ASPI-0425, symbol Device:L_Small
- added L2, L3, L4, L5, L6, L7: 10uH, Inductor_SMD:L_Abracon_ASPI-0425, symbol Device:L_Small
- added Q1: BC857, Package_TO_SOT_SMD:SOT-23, symbol Transistor_BJT:BC857
- added Q2: BC850, Package_TO_SOT_SMD:SOT-23, symbol Transistor_BJT:BC850
- added R10: 6.98K, Resistor_SMD:R_0603_1608Metric, symbol Device:R_Small
- added R11, R14, R15: 110K, Resistor_SMD:R_0603_1608Metric, symbol Device:R_Small
- added R12, R16: 13.3K, Resistor_SMD:R_0603_1608Metric, symbol Device:R_Small
- added R13, R17: 820K, Resistor_SMD:R_0603_1608Metric, symbol Device:R_Small
- added R18: 68.1K, Resistor_SMD:R_0603_1608Metric, symbol Device:R_Small
- added R19: 1.2R, Resistor_SMD:R_0603_1608Metric, symbol Device:R
- added R2: 10R, Resistor_SMD:R_0603_1608Metric, symbol Device:R_Small
- added R5: 18K, Resistor_SMD:R_0603_1608Metric, symbol Device:R_Small
- added R7, R8: 49.9K, Resistor_SMD:R_0603_1608Metric, symbol Device:R_Small
- added R9: 5.1K, Resistor_SMD:R_0603_1608Metric, symbol Device:R_Small
- added RV1: 50K, Potentiometer_THT:Potentiometer_ACP_CA9-V10_Vertical_Hole, symbol Device:R_Potentiometer_Trim
- added TP1, TP10, TP2, TP3, TP4, TP5, TP6, TP7, TP8, TP9: TestPoint, TestPoint:TestPoint_Pad_D1.5mm, symbol Connector:TestPoint
- added U1: TPS61085PW, Package_SO:TSSOP-8_4.4x3mm_P0.65mm, symbol Regulator_Switching:TPS61085PW
- added U2: LM7381, Package_TO_SOT_SMD:SOT-23-5, symbol Amplifier_Operational:NCS325
- added U3: AP3012, Package_TO_SOT_SMD:SOT-23-5, symbol Regulator_Switching:AP3012
- added U4: LMR62014XMF, Package_TO_SOT_SMD:SOT-23-5, symbol Regulator_Switching:LMR62014XMF
- added U5: TPS61040DDC, Package_TO_SOT_SMD:SOT-23-5, symbol Regulator_Switching:TPS61040DDC
- added U6: LM27313XMF, Package_TO_SOT_SMD:SOT-23-5, symbol Regulator_Switching:LM27313XMF
- added U7: TLV61046ADB, Package_TO_SOT_SMD:SOT-23-6, symbol Regulator_Switching:TLV61046ADB
- added U8: TPS61165DBV, Package_TO_SOT_SMD:SOT-23-6, symbol Driver_LED:TPS61165DBV
- C1: renamed from C6; value 10uF/25V -> 2.2uF/50V; footprint (none) -> Capacitor_SMD:C_0805_2012Metric
- C11: renamed from C1; value 2.2uF/25V -> 1uF/50V; footprint (none) -> Capacitor_SMD:C_0805_2012Metric
- C14: renamed from C2; value 10uF/25V -> 2.2uF/50V; footprint (none) -> Capacitor_SMD:C_0805_2012Metric
- C4: renamed from C5; value 2.2uF/25V -> 1uF/50V; footprint (none) -> Capacitor_SMD:C_0805_2012Metric
- C8: renamed from C3; value 0.47uF/25V -> 100nF/50V; footprint (none) -> Capacitor_SMD:C_0603_1608Metric
- D1: renamed from D4; footprint (none) -> Diode_SMD:D_SOD-123
- D6: renamed from D2; footprint (none) -> Diode_SMD:D_SOD-123
- J3: renamed from J1; footprint (none) -> Connector_FFC-FPC:Molex_54132-5033_1x50-1MP_P0.5mm_Horizontal
- R1: renamed from R5; value 47K -> 1K; footprint (none) -> Resistor_SMD:R_0603_1608Metric
- R3: value 0R -> 30K; footprint (none) -> Resistor_SMD:R_0603_1608Metric
- R4: value 220R -> 120K; footprint (none) -> Resistor_SMD:R_0603_1608Metric
- R6: renamed from R2; value 47K -> 1K; footprint (none) -> Resistor_SMD:R_0603_1608Metric
- renumbered D1 to D4
Connections:
- net AVDD: now also R4.1, C10.1, C13.1, D3.1 (K), D5.1 (A), R7.2, TP5.1, U2.5 (V+)
- net DCLK: now also J1.29 (Pin_29), J2.14 (Pin_14)
- net DE: now also J1.28 (Pin_28), J2.42 (Pin_42)
- net DITHB: now also JP15.2 (C)
- net GND: now also J3.MP (MountPin), C10.2, C12.2, C13.2, C15.1, C16.2, C17.2, C18.2, C19.2, C2.2, C21.2, C22.2, C23.2, C24.2, C25.2, C26.2, C27.2, C28.2, C29.2, C3.2, C30.2, C5.1, C7.1, D2.2 (K), J1.1 (Pin_1), J1.13 (Pin_13), J1.25 (Pin_25), J1.37 (Pin_37), J1.7 (Pin_7), J1.MP (MountPin), J2.13 (Pin_13), J2.15 (Pin_15), J2.3 (Pin_3), J2.46 (Pin_46), J2.MP (MountPin), J4.2 (Pin_2), JP12.1 (A), JP14.1 (A), JP15.1 (A), JP16.1 (A), R10.2, R12.2, R14.2, R16.2, R18.2, R19.2, R5.2, R8.2, TP10.1, TP8.1, TP9.1, U1.4 (GND), U2.2 (V-), U3.2 (GND), U4.2 (GND), U5.2 (GND), U6.2 (GND), U7.2 (GND), U8.4 (GND); no longer R1.1, R6.1
- net HSYNC: now also J1.26 (Pin_26), J2.40 (Pin_40)
- net LCD_B0: now also J2.32 (Pin_32)
- net LCD_B1: now also J2.33 (Pin_33)
- net LCD_B2: now also J2.34 (Pin_34)
- net LCD_B3: now also J1.12 (Pin_12), J2.35 (Pin_35)
- net LCD_B4: now also J1.11 (Pin_11), J2.36 (Pin_36)
- net LCD_B5: now also J1.10 (Pin_10), J2.37 (Pin_37)
- net LCD_B6: now also J1.9 (Pin_9), J2.38 (Pin_38)
- net LCD_B7: now also J1.8 (Pin_8), J2.39 (Pin_39)
- net LCD_G0: now also J2.24 (Pin_24)
- net LCD_G1: now also J2.25 (Pin_25)
- net LCD_G2: now also J1.19 (Pin_19), J2.26 (Pin_26)
- net LCD_G3: now also J1.18 (Pin_18), J2.27 (Pin_27)
- net LCD_G4: now also J1.17 (Pin_17), J2.28 (Pin_28)
- net LCD_G5: now also J1.16 (Pin_16), J2.29 (Pin_29)
- net LCD_G6: now also J1.15 (Pin_15), J2.30 (Pin_30)
- net LCD_G7: now also J1.14 (Pin_14), J2.31 (Pin_31)
- net LCD_R0: now also J2.16 (Pin_16)
- net LCD_R1: now also J2.17 (Pin_17)
- net LCD_R2: now also J2.18 (Pin_18)
- net LCD_R3: now also J1.24 (Pin_24), J2.19 (Pin_19)
- net LCD_R4: now also J1.23 (Pin_23), J2.20 (Pin_20)
- net LCD_R5: now also J1.22 (Pin_22), J2.21 (Pin_21)
- net LCD_R6: now also J1.21 (Pin_21), J2.22 (Pin_22)
- net LCD_R7: now also J1.20 (Pin_20), J2.23 (Pin_23)
- net LED_A: now also J1.40 (Pin_40), J2.47 (Pin_47), J2.48 (Pin_48)
- net LED_K: now also J1.38 (Pin_38), J1.39 (Pin_39), J2.49 (Pin_49), J2.50 (Pin_50)
- net L_R_SEL: now also J2.12 (Pin_12), JP12.2 (C)
- net MODE: now also JP16.2 (C)
- net RESET: now also J1.35 (Pin_35), J2.7 (Pin_7)
- net U_D_SEL: now also J2.11 (Pin_11), JP14.2 (C)
- net VCOM: now also C16.1, TP6.1, U2.1, U2.4 (-)
- net VGH: now also C14.1, Q2.2 (E), TP4.1; no longer R3.2
- net VGL: now also C1.1, Q1.2 (E), TP1.1
- net VSYNC: now also J1.27 (Pin_27), J2.41 (Pin_41)
- net at C8.1: now also C6.2, C9.1, JP1.2 (B), R2.2, TP2.1; no longer D4.3 (COM)
- net at C8.2: now also D4.3 (COM)
- net at C4.1: now also R1.2, D2.1 (A), Q1.3 (C); no longer R4.1
- net at D4.1 (A): now also C12.1, D5.2 (K), TP3.1
- net at D4.2 (K): now also C11.1, R6.2, Q2.3 (C), TP7.1
- net DVDD renamed VDD
- net VDD: now also J1.36 (Pin_36), J2.44 (Pin_44), JP13.1 (A)
- new net: C20.1, C23.1, D9.1 (K), JP7.1 (A), R13.1
- new net: C20.2, R13.2, R14.1, U5.3 (FB)
- new net: D7.2 (A), JP2.1 (A), L2.2, U3.1 (SW)
- new net: D6.1 (K), Q2.1 (B), R6.1
- new net: R4.2, R5.1, U1.2 (FB)
- new net: R17.2, R18.1, U7.3 (FB)
- new net: C26.1, D10.1 (K), JP10.1 (A), R15.1
- new net: R15.2, R16.1, U6.3 (FB)
- new net: R8.1, RV1.1
- new net: C29.1, U8.5 (COMP)
- new net: C21.1, D7.1 (K), JP5.1 (A), R9.1
- new net: D3.2 (A), JP1.1 (A), L1.2, R2.1, U1.5 (SW)
- new net: R7.1, RV1.3
- new net: C15.2, RV1.2, U2.3 (+)
- new net: D1.2 (A), Q1.1 (B), R1.1
- new net: C7.2, R3.2
- new net: D9.2 (A), JP4.1 (A), L4.2, U5.1 (SW)
- new net: R3.1, U1.1 (COMP)
- new net: C5.2, U1.8 (SS)
- new net: D10.2 (A), JP8.1 (A), L5.2, U6.1 (SW)
- new net: D11.2 (A), L7.2, U8.3 (SW)
- new net: C6.1, D2.3 (COM)
- new net: D8.2 (A), JP3.1 (A), L3.2, U4.1 (SW)
- new net: R10.1, R9.2, U3.3 (FB)
- new net: JP9.1 (A), L6.2, U7.1 (SW)
- new net: C22.1, D8.1 (K), JP6.1 (A), R11.1
- new net: C27.1, JP11.1 (A), R17.1, U7.5 (VOUT)
- new net: C9.2, D5.3 (COM)
- new net: R11.2, R12.1, U4.3 (FB)
- new net LEDA: C30.1, D11.1 (K)
- new net LEDK: R19.1, U8.6 (FB)
- new net VDD_JMP: JP12.3 (B), JP13.2 (C), JP14.3 (B), JP15.3 (B), JP16.3 (B)
- new net VIN: C17.1, C18.1, C19.1, C2.1, C24.1, C25.1, C28.1, C3.1, J4.1 (Pin_1), JP13.3 (B), L1.1, L2.1, L3.1, L4.1, L5.1, L6.1, L7.1, U1.3 (EN), U1.6 (VIN), U1.7 (FREQ), U3.5 (IN), U4.5 (VIN), U5.5 (VIN), U6.5 (VIN), U7.6 (VI), U8.1 (VIN)
- new net VOUT: JP10.2 (B), JP11.2 (B), JP5.2 (B), JP6.2 (B), JP7.2 (B)
- new net VSW: JP2.2 (B), JP3.2 (B), JP4.2 (B), JP8.2 (B), JP9.2 (B)
- new net ~{SHDN}: U3.4 (~{SHDN}), U4.4 (EN), U5.4 (EN), U6.4 (EN), U7.4 (EN), U8.2 (CTRL)
- no-connect marks 3 -> 22
Other:
- note added: "-7V"
- note added: "10.4V"
- note added: "9.6V"
- note added: "A standard low side resistor of 18 kΩ is typically selected"
- note added: "A value of approximately 13.3 kΩ is recommended for R2"
- note added: "A value of approximately <200K kΩ is recommended for R2"
- note added: "AVDD*2"
- note added: "AVDD*3"
- note added: "For best accuracy, R2 should be kept smaller than 80 kΩ"
- note added: "IR = VFB/ILED VFB=0.2V"
- note added: "LMR62014 and LM27313 is pin to pin and feature compatible They can be substitue each other"
- note added: "R1 = R2 X (VOUT/0.795 − 1)"
- note added: "R1 = R2 X (VOUT/1.23 − 1)"
- note added: "R1 = R2 X (VOUT/1.233 − 1)"
- note added: "R1 = R2 X (VOUT/1.24 − 1)"
- note added: "VOUT = 1.25*(1+R1/R2)"
- note removed: "-7.5V"
- moved on the sheet: C1, C11, C14, C4, C8, D1, D4, D6, J3, R1, R6

Commit message: Changes zener to SOT-23 package, add jobset, generate fabrication file, First release sending to JLCPCB
Parts:
- removed D1, D6: D_Schottky, Diode_SMD:D_SOD-123, symbol Device:D_Schottky
- added D12: BZX84C7V5, Package_TO_SOT_SMD:SOT-23, symbol Diode:BZX84Cxx
- added D13: BZX84C16, Package_TO_SOT_SMD:SOT-23, symbol Diode:BZX84Cxx
- added TP11: TestPoint, TestPoint:TestPoint_Pad_D1.5mm, symbol Connector:TestPoint
- C1, C14: value 2.2uF/50V -> 1uF/50V; JLCPCB Part # (none) -> C28323
- C10, C13, C2: value 10uF -> 10uF/25V; JLCPCB Part # (none) -> C15850
- C11, C12, C4: value 1uF/50V -> 470nF/50V; JLCPCB Part # (none) -> C13967
- C15, C5, C6, C8, C9: JLCPCB Part # (none) -> C14663
- C16: JLCPCB Part # (none) -> C28323
- C3: value 1uF -> 1uF/25V; JLCPCB Part # (none) -> C28323
- C7: JLCPCB Part # (none) -> C710889
- D2, D4, D5: JLCPCB Part # (none) -> C47546
- D3: footprint Diode_SMD:D_SOD-123 -> Diode_SMD:D_SOD-123F; JLCPCB Part # (none) -> C110921
- J1: JLCPCB Part # (none) -> C225713
- J2, J3: footprint Connector_FFC-FPC:Molex_54132-5033_1x50-1MP_P0.5mm_Horizontal -> XF2M_5015_1A:CON50_1X50_DRB_XF2C_TYC; JLCPCB Part # (none) -> C188356
- L1: JLCPCB Part # (none) -> C15269
- Q1: JLCPCB Part # (none) -> C8666
- Q2: JLCPCB Part # (none) -> C80071
- R1: JLCPCB Part # (none) -> C21190
- R2: JLCPCB Part # (none) -> C22859
- R3: JLCPCB Part # (none) -> C22984
- R4: JLCPCB Part # (none) -> C25808
- R5: JLCPCB Part # (none) -> C25810
- R6: value 1K -> 1.6K; JLCPCB Part # (none) -> C22843
- R7, R8: JLCPCB Part # (none) -> C23184
- U1: JLCPCB Part # (none) -> C13505
- U2: value LM7381 -> LM7321; JLCPCB Part # (none) -> C134033
Connections:
- net GND: now also D12.3 (K), D13.1 (A)
- net at Q2.1 (B), R6.1: now also D13.3 (K)
- net at Q1.1 (B), R1.1: now also D12.1 (A)
- net at C4.1, D2.1 (A), Q1.3 (C)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: now also TP11.1
Other:
- moved on the sheet: C12

Commit message: Finished, 1st PCB order to JLCPCB
Parts:
- C15, C5: value 100nF/25V -> 100nF/50V
- C16, C3: value 1uF/25V -> 1uF/50V
